File: Nit.kicad_sch (KiCad schematic)
At the start: 11 parts, among them J1 USB_A, J2 USB_B_Micro, SW1 SW_Push, U1 ATmega328P-P, U2 AMS1117-3.3, U3 CR2013-MI2120, U4 TXB0108PWR, U5 CH559L, Y1 Crystal

Commit message: completed schematic
Parts:
- removed U3: CR2013-MI2120, Display:CR2013-MI2120, symbol Driver_Display:CR2013-MI2120
- added J1: Conn_01x08_Male, symbol Connector:Conn_01x08_Male
- added U3: MSP2807, Connector_PinHeader_2.54mm:PinHeader_1x14_P2.54mm_Vertical, symbol MSP2807:MSP2807
- renumbered J1 to J3
Connections:
- net +3.3V: now also U3.1 (VCC)
- net +5V: now also J1.1 (Pin_1)
- net GND: now also J1.2 (Pin_2), U3.2 (GND)
- net at U4.4 (A3): now also U3.3 (~{CS})
- net at U4.3 (A2): now also U3.5 (D/~{C})
- net at U4.5 (A4): now also U3.6 (MOSI)
- net at U4.7 (A6): now also U3.7 (SCK)
- net at U4.8 (A7): now also U3.8 (LED)
- net at U4.6 (A5): now also U3.9 (MISO)
- net at U1.23 (PC0): now also J1.8 (Pin_8)
- net at U1.24 (PC1): now also J1.7 (Pin_7)
- net at U1.25 (PC2): now also J1.6 (Pin_6)
- net at U1.26 (PC3): now also J1.5 (Pin_5)
- net at U1.27 (PC4): now also J1.4 (Pin_4)
- net at U1.28 (PC5): now also J1.3 (Pin_3)
- net XTAL1: no longer names the net of C1.1, U1.9 (XTAL1/PB6), Y1.1
- net XTAL2: no longer names the net of C2.1, U1.10 (XTAL2/PB7), Y1.2
Other:
- moved on the sheet: C1, C2, J2, J3, Y1

Commit message: Update MSP2807 schematic
Parts:
- J1: footprint (none) -> Connector_PinHeader_2.54mm:PinHeader_1x08_P2.54mm_Horizontal
- U3: footprint Connector_PinHeader_2.54mm:PinHeader_1x14_P2.54mm_Vertical -> Footprint_Library:MSP2807_NaN
Changed lines of the file:
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@@
       (effects (font (size 1.27 1.27)) (justify left))
     )
-    (property "Footprint" "Connector_PinHeader_2.54mm:PinHeader_1x14_P2.54mm_Vertical" (id 2) (at 95.25 151.13 0)
+    (property "Footprint" "Footprint_Library:MSP2807_NaN" (id 2) (at 95.25 151.13 0)
       (effects (font (size 1.27 1.27)) hide)
     )
@@
       (effects (font (size 1.27 1.27)) hide)
     )
+    (pin "")
+    (pin "")
+    (pin "")
+    (pin "")
     (pin "1")
     (pin "10")
@@
     (pin "13")
     (pin "14")
-    (pin "")
-    (pin "")
-    (pin "")
-    (pin "")
     (pin "2")
     (pin "3")
@@
       (effects (font (size 1.27 1.27)) (justify right))
     )
-    (property "Footprint" "" (id 2) (at 80.01 76.2 0)
+    (property "Footprint" "Connector_PinHeader_2.54mm:PinHeader_1x08_P2.54mm_Horizontal" (id 2) (at 80.01 76.2 0)
       (effects (font (size 1.27 1.27)) hide)
     )
@@
     )
     (path "/209d2ef5-7a51-4287-adb6-896daaecb241"
-      (reference "U3") (unit 1) (value "MSP2807") (footprint "Connector_PinHeader_2.54mm:PinHeader_1x14_P2.54mm_Vertical")
+      (reference "U3") (unit 1) (value "MSP2807") (footprint "Footprint_Library:MSP2807_NaN")
     )
     (path "/b92c43ae-e37c-4dc7-a7e8-421ab956ccc8"
